Commit message: UKF compiles and predicts and updates, but the solution is incorrect.There's a bug somewhere in the code that I'm unable to find at the moment.

File: description/urdf/robot_with_sensors.xacro (robot description, xacro)
@@ -12,5 +12,5 @@
       parent_link="${namespace}/base_link"
       imu_topic="demo_imu"
-      mass_imu_sensor="0.00001"
+      mass_imu_sensor="0.015"
       gyroscope_noise_density="0.0003394"
       gyroscope_random_walk="0.000038785"
@@ -22,5 +22,5 @@
       accelerometer_turn_on_bias_sigma="0.1960">
       <inertia ixx="0.00001" ixy="0.0" ixz="0.0" iyy="0.00001" iyz="0.0" izz="0.00001" />
-      <origin xyz="0 0 0" rpy="0 0 0" />
+      <origin xyz="0.015 0 0.0113" rpy="0 0 0" />
     </xacro:imu_sensor_plugin_macro>
   <!-- </xacro:macro> -->

File: description/urdf/robot_with_sensors_ukf.xacro (robot description, xacro)
@@ -12,5 +12,5 @@
       parent_link="${namespace}/base_link"
       imu_topic="demo_imu"
-      mass_imu_sensor="0.00001"
+      mass_imu_sensor="0.015"
       gyroscope_noise_density="0.0003394"
       gyroscope_random_walk="0.000038785"
@@ -22,5 +22,5 @@
       accelerometer_turn_on_bias_sigma="0.1960">
       <inertia ixx="0.00001" ixy="0.0" ixz="0.0" iyy="0.00001" iyz="0.0" izz="0.00001" />
-      <origin xyz="0 0 0" rpy="0 0 0" />
+      <origin xyz="0.015 0 0.0113" rpy="0 0 0" />
     </xacro:imu_sensor_plugin_macro>
   <!-- </xacro:macro> -->
@@ -56,34 +56,3 @@
         <origin xyz="0.0 0.0 0.0" rpy="0.0 0.0 0.0" />
     </xacro:demo_odometry_plugin_macro>
-<!-- Mount a generic odometry sensor without odometry map (working everywhere). -->
-    <xacro:demo_odometry_plugin_macro
-        namespace="${namespace}"
-        plugin_file="librotors_gazebo_odometry_plugin.so"
-        odometry_sensor_suffix="2"
-        parent_link="${namespace}/base_link"
-        pose_topic="odometry_sensor2/pose"
-        pose_with_covariance_topic="odometry_sensor2/pose_with_covariance"
-        position_topic="odometry_sensor2/position"
-        transform_topic="odometry_sensor2/transform"
-        odometry_topic="odometry_sensor2/odometry"
-        parent_frame_id="world"
-        child_frame_id="${namespace}/odometry_sensor2"
-        mass_odometry_sensor="0.00001"
-        measurement_divisor="10"
-        measurement_delay="10"
-        unknown_delay="0.0"
-        noise_normal_position="0.01 0.01 0.01"
-        noise_normal_quaternion="0.017 0.017 0.017"
-        noise_normal_linear_velocity="0 0 0"
-        noise_normal_angular_velocity="0 0 0"
-        noise_uniform_position="0 0 0"
-        noise_uniform_quaternion="0 0 0"
-        noise_uniform_linear_velocity="0 0 0"
-        noise_uniform_angular_velocity="0 0 0"
-        enable_odometry_map="false"
-        odometry_map=""
-        image_scale="">
-        <inertia ixx="0.00001" ixy="0.0" ixz="0.0" iyy="0.00001" iyz="0.0" izz="0.00001" /> <!-- [kg m^2] [kg m^2] [kg m^2] [kg m^2] [kg m^2] [kg m^2] -->
-        <origin xyz="0.03 -0.07 0.1" rpy="0.2 -0.1 0.3" />
-    </xacro:demo_odometry_plugin_macro>
 </robot>
